File: hardware/cellular_modem.kicad_sch (KiCad schematic)
At the start: 33 parts, among them J2 0786463001, J3 RF2-04A-T-00-50-G, Q4 2N7002, Q5 2N7002, U3 BC65PB-04-STD, U4 TPS61200DRC

Commit message: begin stm32 implementation and remove battery charger for simplicity
Parts:
- renumbered U3 to U4, U4 to U5
Changed lines of the file:
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@@
 		(dnp no)
 		(fields_autoplaced yes)
-		(property "Reference" "U3"
+		(property "Reference" "U4"
 			(at 177.8 19.05 0)
 			(effects
@@
 			(project ""
 				(path "/34886a96-89cd-4fc5-ba47-006a1318e849/efb4cfd9-4abf-484f-b828-d075dddb773a"
-					(reference "U3")
+					(reference "U4")
 					(unit 1)
 				)
@@
 		(dnp no)
 		(fields_autoplaced yes)
-		(property "Reference" "U4"
+		(property "Reference" "U5"
 			(at 46.99 26.67 0)
 			(effects
@@
 			(project ""
 				(path "/34886a96-89cd-4fc5-ba47-006a1318e849/efb4cfd9-4abf-484f-b828-d075dddb773a"
-					(reference "U4")
-					(unit 1)
-				)
+					(reference "U5")
+					(unit 1)
+				)

Commit message: refactor power delivery to support higher current loads
Connections:
- net +3.3V renamed VBUS
Changed lines of the file:
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@@
 	(wire
 		(pts
-			(xy 19.05 33.02) (xy 19.05 34.29)
+			(xy 19.05 31.75) (xy 19.05 34.29)
 		)
 		(stroke
@@
 	)
 	(symbol
+		(lib_id "power:VBUS")
+		(at 19.05 31.75 0)
+		(unit 1)
+		(exclude_from_sim no)
+		(in_bom yes)
+		(on_board yes)
+		(dnp no)
+		(property "Reference" "#PWR01"
+			(at 19.05 35.56 0)
+			(effects
+				(font
+					(size 1.27 1.27)
+				)
+				(hide yes)
+			)
+		)
+		(property "Value" "VBUS"
+			(at 19.05 27.94 0)
+			(effects
+				(font
+					(size 1.27 1.27)
+				)
+			)
+		)
+		(property "Footprint" ""
+			(at 19.05 31.75 0)
+			(effects
+				(font
+					(size 1.27 1.27)
+				)
+				(hide yes)
+			)
+		)
+		(property "Datasheet" ""
+			(at 19.05 31.75 0)
+			(effects
+				(font
+					(size 1.27 1.27)
+				)
+				(hide yes)
+			)
+		)
+		(property "Description" "Power symbol creates a global label with name \"VBUS\""
+			(at 19.05 31.75 0)
+			(effects
+				(font
+					(size 1.27 1.27)
+				)
+				(hide yes)
+			)
+		)
+		(pin "1"
+		)
+		(instances
+			(project ""
+				(path "/34886a96-89cd-4fc5-ba47-006a1318e849/efb4cfd9-4abf-484f-b828-d075dddb773a"
+					(reference "#PWR01")
+					(unit 1)
+				)
+			)
+		)
+	)
+	(symbol
 		(lib_id "Device:R")
 		(at 35.56 85.09 90)
@@
 					(unit 1)
 				)
-			)
-		)
-	)
-	(symbol
-		(lib_id "power:+3.3V")
-		(at 19.05 33.02 0)
-		(unit 1)
-		(exclude_from_sim no)
-		(in_bom yes)
-		(on_board yes)
-		(dnp no)
-		(fields_autoplaced yes)
-		(property "Reference" "#PWR05"
-			(at 19.05 36.83 0)
-			(effects
-				(font
-					(size 1.27 1.27)
-				)
-				(hide yes)
-			)
-		)
-		(property "Value" "+3.3V"
-			(at 19.05 27.94 0)
-			(effects
-				(font
-					(size 1.27 1.27)
-				)
-			)
-		)
-		(property "Footprint" ""
-			(at 19.05 33.02 0)
-			(effects
-				(font
-					(size 1.27 1.27)
-				)
-				(hide yes)
-			)
-		)
-		(property "Datasheet" ""
-			(at 19.05 33.02 0)
-			(effects
-				(font
-					(size 1.27 1.27)
-				)
-				(hide yes)
-			)
-		)
-		(property "Description" "Power symbol creates a global label with name \"+3.3V\""
-			(at 19.05 33.02 0)
-			(effects
-				(font
-					(size 1.27 1.27)
-				)
-				(hide yes)
-			)
-		)
-		(pin "1"
-		)
-		(instances
-			(project ""
-				(path "/34886a96-89cd-4fc5-ba47-006a1318e849/efb4cfd9-4abf-484f-b828-d075dddb773a"
-					(reference "#PWR05")
-					(unit 1)
-				)
